File: main/keycluster-main.kicad_pcb (KiCad board)
At the start: 2 copper layers, 45.1 x 52.6 mm, 33 parts, among them P2 CONN_5, P7 CONN_10, P8 CONN_7, SW1 S01_Socket, SW2 S01_Socket, SW3 S01_Socket, SW4 CMI126603D08, SW6 CMI126603D08, U1 MKL03Z32VFK4, U2 IS31FL3199, U4 ESD

Commit message: Completed routing.
Parts:
- moved R1 17.8 mm to (157.6, 124.0)
- moved C3 1.51 mm to (150.6, 107.4), turned to 240 degrees
Connections:
- P8 pad : (no net) -> GND
- U2 pad 10: Net-(D3-Pad3) -> Net-(D3-Pad1)
- U2 pad 11: Net-(D3-Pad1) -> Net-(D3-Pad2)
- U2 pad 12: Net-(D3-Pad2) -> Net-(D3-Pad3)
Routing:
- net Net-(R5-Pad1): track 12.4 -> 42.0 mm, vias 1 -> 2
- net GND: track 41.4 -> 54.6 mm, vias 13 -> 17
- net /RESET: track 21.4 -> 29.0 mm, vias 2 -> 4
- net +3V3: track 52.2 -> 57.8 mm
- net Net-(D3-Pad3): track 23.2 -> 25.6 mm, vias 1 -> 2
- net /SWDIO: track 20.0 -> 22.4 mm
- net /TB_DOWN: track 29.3 -> 27.5 mm
- net /SCL: track 76.6 -> 74.7 mm
- net /SW4: track 44.3 -> 42.8 mm
- net /SW5: track 27.6 -> 29.0 mm
- net +5V: track 125.9 -> 124.6 mm
- net /TB_LEFT: track 39.4 -> 40.6 mm
- net Net-(D3-Pad1): track 13.8 -> 14.9 mm, vias 2 -> 0
- net /SWDCLK: track 18.8 -> 18.0 mm
- net /TB_RIGHT: track 24.3 -> 25.0 mm
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